File: 7.0/projects/Regulateur_tension/regulateur_tension-backup_ok_fin19-10-2024/regulateur_tension.kicad_pcb (KiCad board)
At the start: 2 copper layers, 81.3 x 50.8 mm, 11 parts

Commit message: checkpoint-OK-multiple-piste-trace-1.5mm
Changed lines of the file:
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@@
 		(start 22.98 20.32)
 		(end 34.41 20.32)
-		(width 1.5)
+		(width 1)
 		(layer "B.Cu")
 		(net 1)
@@
 		(start 78.86 22.98)
 		(end 78.86 26.55)
-		(width 1.5)
+		(width 1)
 		(layer "B.Cu")
 		(net 1)
@@
 		(start 58.42 20.44)
 		(end 76.32 20.44)
-		(width 1.5)
+		(width 1)
 		(layer "B.Cu")
 		(net 1)
@@
 		(start 43.3 20.44)
 		(end 58.42 20.44)
-		(width 1.5)
+		(width 1)
 		(layer "B.Cu")
 		(net 1)
@@
 		(start 34.41 20.32)
 		(end 38.1 24.01)
-		(width 1.5)
+		(width 1)
 		(layer "B.Cu")
 		(net 1)
@@
 		(start 17.78 25.52)
 		(end 22.98 20.32)
-		(width 1.5)
+		(width 1)
+		(layer "B.Cu")
+		(net 1)
+	)
+	(segment
+		(start 21.47 54.49)
+		(end 17.78 50.8)
+		(width 1)
+		(layer "B.Cu")
+		(net 1)
+	)
+	(segment
+		(start 22.98 54.49)
+		(end 21.47 54.49)
+		(width 1)
 		(layer "B.Cu")
 		(net 1)
@@
 		(start 76.32 20.44)
 		(end 78.86 22.98)
-		(width 1.5)
-		(layer "B.Cu")
-		(net 1)
-	)
-	(segment
-		(start 22.98 54.49)
-		(end 21.47 54.49)
-		(width 1.5)
+		(width 1)
 		(layer "B.Cu")
 		(net 1)
@@
 	)
 	(segment
-		(start 21.47 54.49)
-		(end 17.78 50.8)
-		(width 1.5)
-		(layer "B.Cu")
-		(net 1)
-	)
-	(segment
 		(start 39.49 24.01)
 		(end 43.18 20.32)
-		(width 1.5)
+		(width 1)
 		(layer "B.Cu")
 		(net 1)
@@
 		(start 17.78 50.8)
 		(end 17.78 25.52)
-		(width 1.5)
+		(width 1)
 		(layer "B.Cu")
 		(net 1)
@@
 		(start 78.94 48.06)
 		(end 78.94 45.72)
-		(width 1.5)
+		(width 1)
 		(layer "B.Cu")
 		(net 2)
@@
 		(start 53.34 36.71)
 		(end 58.42 31.63)
-		(width 1.5)
+		(width 1)
 		(layer "B.Cu")
 		(net 2)
@@
 		(start 58.42 31.63)
 		(end 58.42 27.94)
-		(width 1.5)
+		(width 1)
 		(layer "B.Cu")
 		(net 2)
@@
 		(start 83.94 45.72)
 		(end 91.56 38.1)
-		(width 1.5)
+		(width 1)
 		(layer "B.Cu")
 		(net 2)
@@
 		(start 49.53 27.94)
 		(end 58.42 27.94)
-		(width 1.5)
+		(width 1)
 		(layer "B.Cu")
 		(net 2)
@@
 		(start 53.34 54.49)
 		(end 72.51 54.49)
-		(width 1.5)
+		(width 1)
 		(layer "B.Cu")
 		(net 2)
@@
 		(start 45.6 24.01)
 		(end 49.53 27.94)
-		(width 1.5)
+		(width 1)
 		(layer "B.Cu")
 		(net 2)
@@
 		(start 72.51 54.49)
 		(end 78.94 48.06)
-		(width 1.5)
+		(width 1)
 		(layer "B.Cu")
 		(net 2)
@@
 		(start 53.34 54.49)
 		(end 53.34 36.71)
-		(width 1.5)
+		(width 1)
 		(layer "B.Cu")
 		(net 2)
@@
 		(start 83.94 45.72)
 		(end 78.94 45.72)
-		(width 1.5)
+		(width 1)
 		(layer "B.Cu")
 		(net 2)
@@
 		(start 22.98 34.17)
 		(end 22.98 30.48)
-		(width 1.5)
+		(width 1)
 		(layer "B.Cu")
 		(net 3)
@@
 		(start 38.22 39.25)
 		(end 40.76 36.71)
-		(width 1.5)
+		(width 1)
 		(layer "B.Cu")
 		(net 3)
@@
 		(start 30.6 39.25)
 		(end 28.06 39.25)
-		(width 1.5)
+		(width 1)
 		(layer "B.Cu")
 		(net 3)
@@
 		(start 40.76 36.71)
 		(end 43.18 36.71)
-		(width 1.5)
+		(width 1)
 		(layer "B.Cu")
 		(net 3)
@@
 		(start 28.06 39.25)
 		(end 22.98 34.17)
-		(width 1.5)
+		(width 1)
 		(layer "B.Cu")
 		(net 3)
@@
 		(start 30.6 39.25)
 		(end 38.22 39.25)
-		(width 1.5)
+		(width 1)
 		(layer "B.Cu")
 		(net 3)
@@
 		(start 33.14 54.49)
 		(end 33.14 46.79)
-		(width 1.5)
+		(width 1)
 		(layer "B.Cu")
 		(net 4)
@@
 		(start 33.14 46.79)
 		(end 30.6 44.25)
-		(width 1.5)
+		(width 1)
 		(layer "B.Cu")
 		(net 4)
@@
 		(start 33.14 54.49)
 		(end 43.18 54.49)
-		(width 1.5)
+		(width 1)
 		(layer "B.Cu")
 		(net 4)
@@
 		(start 76.32 26.55)
 		(end 76.32 35.44)
-		(width 1.5)
+		(width 1)
 		(layer "B.Cu")
 		(net 5)
@@
 		(start 82.67 31.63)
 		(end 78.74 35.56)
-		(width 1.5)
+		(width 1)
 		(layer "B.Cu")
 		(net 5)
@@
 		(start 78.74 35.56)
 		(end 76.2 35.56)
-		(width 1.5)
+		(width 1)
 		(layer "B.Cu")
 		(net 5)
@@
 		(start 91.56 31.63)
 		(end 82.67 31.63)
-		(width 1.5)
+		(width 1)
 		(layer "B.Cu")
 		(net 5)
@@
 		(start 71.12 35.56)
 		(end 71.12 29.21)
-		(width 1.5)
+		(width 1)
 		(layer "B.Cu")
 		(net 6)
@@
 		(start 71.12 43.18)
 		(end 71.12 35.56)
-		(width 1.5)
+		(width 1)
 		(layer "B.Cu")
 		(net 6)
@@
 		(start 71.12 29.21)
 		(end 73.78 26.55)
-		(width 1.5)
+		(width 1)
 		(layer "B.Cu")
 		(net 6)
@@
 		(start 73.94 45.72)
 		(end 71.4 43.18)
-		(width 1.5)
-		(layer "B.Cu")
-		(net 6)
+		(width 1)
+		(layer "B.Cu")
+		(net 6)
