File: 7.0/projects/Regulateur_tension/regulateur_tension/regulateur_tension.kicad_pcb (KiCad board)
At the start: 2 copper layers, 81.3 x 50.8 mm, 11 parts

Commit message: final-final
Parts:
- D1, D2, D3, D4: value 1N4001 -> 1N4007
- INPUT_AC1: value ~ -> IN_AC
- R2: value 570 -> 654
Changed lines of the file:
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@@
 			(drillshape 0)
 			(scaleselection 1)
-			(outputdirectory "gerber-regula-26-08-2024-v3_back/")
+			(outputdirectory "gerber-regul-22-10-2024-v7.0/")
 		)
 	)
@@
 			)
 		)
-		(property "Datasheet" ""
+		(property "Datasheet" "https://www.reboul.fr/storage/00008823.pdf"
 			(at 0 0 0)
 			(unlocked yes)
@@
 			)
 		)
-		(property "Value" "570"
+		(property "Value" "654"
 			(at 5.08 -14.96 90)
 			(layer "F.Fab")
@@
 			)
 		)
-		(property "Datasheet" ""
+		(property "Datasheet" "https://www.farnell.com/datasheets/3667870.pdf"
 			(at 0 0 -90)
 			(unlocked yes)
@@
 			)
 		)
-		(property "Value" "1N4001"
+		(property "Value" "1N4007"
 			(at 5.08 2.47 0)
 			(layer "F.Fab")
@@
 			)
 		)
-		(property "Datasheet" ""
+		(property "Datasheet" "https://www.farnell.com/datasheets/2866634.pdf"
 			(at 0 0 90)
 			(unlocked yes)
@@
 			)
 		)
-		(property "Value" "1N4001"
+		(property "Value" "1N4007"
 			(at 5.08 2.47 0)
 			(layer "F.Fab")
@@
 			)
 		)
-		(property "Datasheet" ""
+		(property "Datasheet" "https://www.reboul.fr/storage/00008823.pdf"
 			(at 0 0 -90)
 			(unlocked yes)
@@
 			)
 		)
-		(property "Value" "1N4001"
+		(property "Value" "1N4007"
 			(at 5.08 -4.96 90)
 			(layer "F.Fab")
@@
 			)
 		)
-		(property "Value" "1N4001"
+		(property "Value" "1N4007"
 			(at 5.08 2.47 0)
 			(layer "F.Fab")
@@
 			)
 		)
-		(property "Value" "~"
+		(property "Value" "IN_AC"
 			(at 2.5 5.06 90)
 			(layer "F.Fab")
@@
 			)
 		)
-		(property "Datasheet" ""
+		(property "Datasheet" "https://www.farnell.com/datasheets/2866634.pdf"
 			(at 0 0 -90)
 			(unlocked yes)
@@
 			)
 		)
-		(property "Sim.Device" "V"
-			(at 0 0 -90)
-			(unlocked yes)
-			(layer "F.Fab")
-			(hide yes)
-			(effects
-				(font
-					(size 1 1)
-					(thickness 0.15)
-				)
-			)
-		)
-		(property "Sim.Type" "SIN"
-			(at 0 0 -90)
-			(unlocked yes)
-			(layer "F.Fab")
-			(hide yes)
-			(effects
-				(font
-					(size 1 1)
-					(thickness 0.15)
-				)
-			)
-		)
-		(property "Sim.Params" "dc=0 ampl=10 f=0 td=0 theta=0 phase=0 ac=10"
-			(at 0 0 -90)
-			(unlocked yes)
-			(layer "F.Fab")
-			(hide yes)
-			(effects
-				(font
-					(size 1 1)
-					(thickness 0.15)
-				)
-			)
-		)
-		(property "Sim.Pins" "1=+ 2=-"
-			(at 0 0 -90)
-			(unlocked yes)
-			(layer "F.Fab")
-			(hide yes)
-			(effects
-				(font
-					(size 1 1)
-					(thickness 0.15)
-				)
-			)
-		)
 		(property ki_fp_filters "Connector*:*_1x??_*")
 		(sheetname "Racine")
@@
 			)
 		)
-		(property "Datasheet" ""
+		(property "Datasheet" "https://www.farnell.com/datasheets/3436052.pdf"
 			(at 0 0 180)
 			(unlocked yes)
