File: 7.0/projects/Regulateur_tension/regulateur_tension/regulateur_tension.kicad_sch (KiCad schematic)
At the start: 11 parts

Commit message: final-final
Parts:
- D1, D2, D3, D4: value 1N4001 -> 1N4007
- INPUT_AC1: value ${SIM.PARAMS} -> IN_AC
- R2: value 570 -> 654
Changed lines of the file:
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@@
 			)
 		)
-		(property "Value" "${SIM.PARAMS}"
+		(property "Value" "IN_AC"
 			(at 46.99 66.0399 0)
 			(effects
@@
 			)
 		)
-		(property "Datasheet" "~"
+		(property "Datasheet" "https://www.farnell.com/datasheets/2866634.pdf"
 			(at 49.53 63.5 0)
 			(effects
@@
 			)
 		)
-		(property "Datasheet" "~"
+		(property "Datasheet" "https://www.reboul.fr/storage/00008823.pdf"
 			(at 91.44 63.5 0)
 			(effects
@@
 		(fields_autoplaced yes)
 		(property "Reference" "D3"
-			(at 63.5 59.69 90)
-			(effects
-				(font
-					(size 1.27 1.27)
-				)
-				(justify left)
-			)
-		)
-		(property "Value" "1N4001"
-			(at 63.5 62.23 90)
+			(at 63.5 59.6899 90)
+			(effects
+				(font
+					(size 1.27 1.27)
+				)
+				(justify left)
+			)
+		)
+		(property "Value" "1N4007"
+			(at 63.5 62.2299 90)
 			(effects
 				(font
@@
 	)
 	(symbol
+		(lib_name "C_Polarized_1")
 		(lib_id "Device:C_Polarized")
 		(at 104.14 64.77 0)
@@
 			)
 		)
-		(property "Datasheet" "~"
+		(property "Datasheet" "https://www.reboul.fr/storage/00008823.pdf"
 			(at 104.14 64.77 0)
 			(effects
@@
 			)
 		)
-		(property "Value" "1N4001"
+		(property "Value" "1N4007"
 			(at 69.85 43.18 0)
 			(effects
@@
 			)
 		)
-		(property "Value" "1N4001"
+		(property "Value" "1N4007"
 			(at 81.28 64.7699 90)
 			(effects
@@
 			)
 		)
-		(property "Datasheet" "~"
+		(property "Datasheet" "https://www.farnell.com/datasheets/3436052.pdf"
 			(at 146.05 63.5 0)
 			(effects
@@
 			)
 		)
-		(property "Datasheet" "~"
+		(property "Datasheet" "https://www.farnell.com/datasheets/2866634.pdf"
 			(at 166.37 62.23 0)
 			(effects
@@
 			)
 		)
-		(property "Value" "1N4001"
+		(property "Value" "1N4007"
 			(at 82.55 73.66 0)
 			(effects
@@
 			)
 		)
-		(property "Value" "570"
+		(property "Value" "654"
 			(at 124.46 74.9299 0)
 			(effects
@@
 			)
 		)
-		(property "Datasheet" "~"
+		(property "Datasheet" "https://www.farnell.com/datasheets/3667870.pdf"
 			(at 127 73.66 0)
 			(effects
