File: 7.0/projects/Transformateur/transformateur_circuit/transformateur_circuit.kicad_pcb (KiCad board)
At the start: 2 copper layers, 96.5 x 45.7 mm, 5 parts

Commit message: adding  timmer 55 project
Parts:
- added F1: 500m, Resistor_THT:R_Axial_Power_L20.0mm_W6.4mm_P22.40mm, F.Cu at (152.4, 169.4)
- added F1: 500m, Resistor_THT:R_Axial_Power_L20.0mm_W6.4mm_P22.40mm, F.Cu at (151.4, 115.8)
- added F1: 500m, Resistor_THT:R_Axial_Power_L20.0mm_W6.4mm_P22.40mm, F.Cu at (46.7, 115.8)
- added F1: 500m, Resistor_THT:R_Axial_Power_L20.0mm_W6.4mm_P22.40mm, F.Cu at (150.4, 56.9)
- added F1: 500m, Resistor_THT:R_Axial_Power_L20.0mm_W6.4mm_P22.40mm, F.Cu at (47.8, 169.4)
- added F2: 500m, Resistor_THT:R_Axial_Power_L20.0mm_W6.4mm_P22.40mm, F.Cu at (206.2, 50.3)
- added F2: 500m, Resistor_THT:R_Axial_Power_L20.0mm_W6.4mm_P22.40mm, F.Cu at (103.6, 162.8)
- added F2: 500m, Resistor_THT:R_Axial_Power_L20.0mm_W6.4mm_P22.40mm, F.Cu at (208.3, 162.8)
- added F2: 500m, Resistor_THT:R_Axial_Power_L20.0mm_W6.4mm_P22.40mm, F.Cu at (207.3, 109.2)
- added F2: 500m, Resistor_THT:R_Axial_Power_L20.0mm_W6.4mm_P22.40mm, F.Cu at (102.6, 109.2)
- added INPUT1: INPUT_230V_AC, TerminalBlock_MetzConnect:TerminalBlock_MetzConnect_Type094_RT03502HBLU_1x02_P5.00mm_Horizontal, F.Cu at (137.7, 36.6)
- added INPUT1: INPUT_230V_AC, TerminalBlock_MetzConnect:TerminalBlock_MetzConnect_Type094_RT03502HBLU_1x02_P5.00mm_Horizontal, F.Cu at (139.7, 149.1)
- added INPUT1: INPUT_230V_AC, TerminalBlock_MetzConnect:TerminalBlock_MetzConnect_Type094_RT03502HBLU_1x02_P5.00mm_Horizontal, F.Cu at (138.7, 95.5)
- added INPUT1: INPUT_230V_AC, TerminalBlock_MetzConnect:TerminalBlock_MetzConnect_Type094_RT03502HBLU_1x02_P5.00mm_Horizontal, F.Cu at (34.0, 95.5)
- added INPUT1: INPUT_230V_AC, TerminalBlock_MetzConnect:TerminalBlock_MetzConnect_Type094_RT03502HBLU_1x02_P5.00mm_Horizontal, F.Cu at (35.1, 149.1)
- added OUTPUT1: OUTPUT_12_AC, TerminalBlock_MetzConnect:TerminalBlock_MetzConnect_Type094_RT03502HBLU_1x02_P5.00mm_Horizontal, F.Cu at (221.0, 161.7)
- added OUTPUT1: OUTPUT_12_AC, TerminalBlock_MetzConnect:TerminalBlock_MetzConnect_Type094_RT03502HBLU_1x02_P5.00mm_Horizontal, F.Cu at (218.9, 49.2)
- added OUTPUT1: OUTPUT_12_AC, TerminalBlock_MetzConnect:TerminalBlock_MetzConnect_Type094_RT03502HBLU_1x02_P5.00mm_Horizontal, F.Cu at (115.3, 108.1)
- added OUTPUT1: OUTPUT_12_AC, TerminalBlock_MetzConnect:TerminalBlock_MetzConnect_Type094_RT03502HBLU_1x02_P5.00mm_Horizontal, F.Cu at (116.3, 161.7)
- added OUTPUT1: OUTPUT_12_AC, TerminalBlock_MetzConnect:TerminalBlock_MetzConnect_Type094_RT03502HBLU_1x02_P5.00mm_Horizontal, F.Cu at (220.0, 108.1)
- added TR1: TRANSF, Transformer_THT:Transformer_Breve_TEZ-38x45, F.Cu at (63.2, 169.2)
- added TR1: TRANSF, Transformer_THT:Transformer_Breve_TEZ-38x45, F.Cu at (167.8, 169.2)
- added TR1: TRANSF, Transformer_THT:Transformer_Breve_TEZ-38x45, F.Cu at (62.2, 115.6)
- added TR1: TRANSF, Transformer_THT:Transformer_Breve_TEZ-38x45, F.Cu at (166.8, 115.6)
- added TR1: TRANSF, Transformer_THT:Transformer_Breve_TEZ-38x45, F.Cu at (165.8, 56.7)
- moved F2 50.1 mm to (102.6, 50.3)
- moved F1 50.1 mm to (46.7, 56.9)
- moved INPUT1 50.1 mm to (34.0, 36.6)
- moved OUTPUT1 50.1 mm to (115.3, 49.2)
- moved TR1 50.1 mm to (62.2, 56.7)
Routing:
- net Net-(INPUT1-Pin_2): track 62.5 -> 375.3 mm
- net Net-(OUTPUT1-Pin_2): track 53.3 -> 319.9 mm
- net Net-(F2-Pad2): track 28.4 -> 170.3 mm
- net Net-(F1-Pad1): track 15.5 -> 93.1 mm
- net Net-(INPUT1-Pin_1): track 13.6 -> 81.4 mm
- net Net-(OUTPUT1-Pin_1): track 13.2 -> 79.0 mm
Other:
- board size 96.5 x 45.7 mm -> 202.2 x 158.2 mm
