File: 7.0/projects/Transformateur/transformateur_circuit/transformateur_circuit.kicad_sch (KiCad schematic)
At the start: 5 parts

Commit message: adding  timmer 55 project
Other:
- company: (none) -> Solare-elec
- title: (none) -> Transformateur
Changed lines of the file:
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@@
 	(generator_version "8.0")
 	(paper "A4")
+	(title_block
+		(title "Transformateur")
+		(date "2024-11-03")
+		(rev "0.0.1")
+		(company "Solare-elec")
+	)
 	(wire
 		(pts
