File: 7.0/projects/ADC_conversion/ADC_conversion/ADC_conversion.kicad_sch (KiCad schematic)
At the start: 4 parts, among them U1 ATmega32-16P

Commit message: adding sample projects
Parts:
- added R2: R, symbol Device:R
- added R_POTEN1: 2kOhm, symbol Device:R_Potentiometer
- added SRC_DC1, SRC_DC2: 5V, symbol Device:Battery_Cell
- added U2: ATmega32-16P, Package_DIP:DIP-40_W15.24mm, symbol MCU_Microchip_ATmega:ATmega32-16P
- R1: value R -> 100
- R_POTEN: value 2kOhm -> 1kOhm
Connections:
- net AVCC: now also SRC_DC2.1 (+), U2.10 (VCC), U2.30 (AVCC)
- net GND: now also R_POTEN1.2, SRC_DC1.2 (-), SRC_DC2.2 (-), U2.11 (GND), U2.31 (GND)
- net PA1: now also R2.1, R_POTEN1.1, U2.39 (PA1)
- new net: R2.2, SRC_DC1.1 (+)
Other:
- note added: "MONTAGE SOURCE MULTIPLE DE TENSION"
- note added: "MONTAGE SOURCE UNIQUE DE TENSION"
- moved on the sheet: R1, R_POTEN, SRC_DC, U1
