File: 7.0/projects/Ecran_LCD_16_02/Ecran_LCD_16_02.kicad_sch (KiCad schematic)
At the start: 4 parts

Commit message: adding somme kicad corrections
Connections:
- net GND: no longer R1.2
- net VDD: now reaches A1.5 (+5V), DS1.2 (VDD), RV1.3
- net VDD: now also R1.2
Other:
- moved on the sheet: R1
Changed lines of the file:
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@@
 	)
 	(junction
-		(at 73.66 100.33)
+		(at 90.17 100.33)
 		(diameter 0)
 		(color 0 0 0 0)
@@
 		(color 0 0 0 0)
 	)
-	(junction
-		(at 80.01 100.33)
-		(diameter 0)
-		(color 0 0 0 0)
-	)
-	(wire
-		(pts
-			(xy 73.66 100.33) (xy 80.01 100.33)
-		)
-		(stroke
-			(width 0)
-			(type default)
-		)
-	)
 	(wire
 		(pts
@@
 	(wire
 		(pts
-			(xy 73.66 80.01) (xy 73.66 72.39)
+			(xy 74.93 76.2) (xy 74.93 72.39)
 		)
 		(stroke
@@
 	(wire
 		(pts
-			(xy 138.43 109.22) (xy 138.43 110.49)
-		)
-		(stroke
-			(width 0)
-			(type default)
-		)
-	)
-	(wire
-		(pts
 			(xy 102.87 64.77) (xy 100.33 64.77)
 		)
@@
 	(wire
 		(pts
+			(xy 74.93 83.82) (xy 74.93 87.63)
+		)
+		(stroke
+			(width 0)
+			(type default)
+		)
+	)
+	(wire
+		(pts
 			(xy 160.02 83.82) (xy 162.56 83.82)
 		)
@@
 	(wire
 		(pts
-			(xy 73.66 72.39) (xy 80.01 72.39)
-		)
-		(stroke
-			(width 0)
-			(type default)
-		)
-	)
-	(wire
-		(pts
-			(xy 73.66 87.63) (xy 73.66 100.33)
+			(xy 74.93 72.39) (xy 80.01 72.39)
 		)
 		(stroke
@@
 		)
 	)
+	(global_label "VDD"
+		(shape input)
+		(at 90.17 49.53 180)
+		(fields_autoplaced yes)
+		(effects
+			(font
+				(size 1.27 1.27)
+			)
+			(justify right)
+		)
+		(property "Intersheetrefs" "${INTERSHEET_REFS}"
+			(at 83.5562 49.53 0)
+			(effects
+				(font
+					(size 1.27 1.27)
+				)
+				(justify right)
+				(hide yes)
+			)
+		)
+	)
 	(global_label "UNO_PIN5"
 		(shape input)
@@
 				)
 				(justify left)
+				(hide yes)
+			)
+		)
+	)
+	(global_label "VDD"
+		(shape input)
+		(at 74.93 87.63 270)
+		(fields_autoplaced yes)
+		(effects
+			(font
+				(size 1.27 1.27)
+			)
+			(justify right)
+		)
+		(property "Intersheetrefs" "${INTERSHEET_REFS}"
+			(at 74.93 94.2438 90)
+			(effects
+				(font
+					(size 1.27 1.27)
+				)
+				(justify right)
 				(hide yes)
 			)
@@
 	(symbol
 		(lib_id "power:GND")
-		(at 138.43 110.49 0)
+		(at 138.43 109.22 0)
 		(unit 1)
 		(exclude_from_sim no)
@@
 		(on_board yes)
 		(dnp no)
-		(fields_autoplaced yes)
 		(property "Reference" "#PWR02"
-			(at 138.43 116.84 0)
+			(at 138.43 115.57 0)
 			(effects
 				(font
@@
 		)
 		(property "Value" "GND"
-			(at 138.43 115.57 0)
+			(at 134.874 110.998 0)
 			(effects
 				(font
@@
 		)
 		(property "Footprint" ""
-			(at 138.43 110.49 0)
+			(at 138.43 109.22 0)
 			(effects
 				(font
@@
 		)
 		(property "Datasheet" ""
-			(at 138.43 110.49 0)
+			(at 138.43 109.22 0)
 			(effects
 				(font
@@
 		)
 		(property "Description" "Power symbol creates a global label with name \"GND\" , ground"
-			(at 138.43 110.49 0)
+			(at 138.43 109.22 0)
 			(effects
 				(font
@@
 	)
 	(symbol
-		(lib_id "power:GND")
-		(at 73.66 100.33 0)
-		(unit 1)
-		(exclude_from_sim no)
-		(in_bom yes)
-		(on_board yes)
-		(dnp no)
-		(fields_autoplaced yes)
-		(property "Reference" "#PWR01"
-			(at 73.66 106.68 0)
-			(effects
-				(font
-					(size 1.27 1.27)
-				)
-				(hide yes)
-			)
-		)
-		(property "Value" "GND"
-			(at 73.66 105.41 0)
-			(effects
-				(font
-					(size 1.27 1.27)
-				)
-			)
-		)
-		(property "Footprint" ""
-			(at 73.66 100.33 0)
-			(effects
-				(font
-					(size 1.27 1.27)
-				)
-				(hide yes)
-			)
-		)
-		(property "Datasheet" ""
-			(at 73.66 100.33 0)
-			(effects
-				(font
-					(size 1.27 1.27)
-				)
-				(hide yes)
-			)
-		)
-		(property "Description" "Power symbol creates a global label with name \"GND\" , ground"
-			(at 73.66 100.33 0)
-			(effects
-				(font
-					(size 1.27 1.27)
-				)
-				(hide yes)
-			)
-		)
-		(pin "1"
-		)
-		(instances
-			(project ""
-				(path "/da3a0145-d0f3-4b31-b746-e8b9b9ecb582"
-					(reference "#PWR01")
-					(unit 1)
-				)
-			)
-		)
-	)
-	(symbol
 		(lib_id "Device:R_Potentiometer")
 		(at 166.37 83.82 180)
@@
 				(path "/da3a0145-d0f3-4b31-b746-e8b9b9ecb582"
 					(reference "RV1")
+					(unit 1)
+				)
+			)
+		)
+	)
+	(symbol
+		(lib_id "power:GND")
+		(at 90.17 100.33 0)
+		(unit 1)
+		(exclude_from_sim no)
+		(in_bom yes)
+		(on_board yes)
+		(dnp no)
+		(property "Reference" "#PWR01"
+			(at 90.17 106.68 0)
+			(effects
+				(font
+					(size 1.27 1.27)
+				)
+				(hide yes)
+			)
+		)
+		(property "Value" "GND"
+			(at 86.614 102.108 0)
+			(effects
+				(font
+					(size 1.27 1.27)
+				)
+			)
+		)
+		(property "Footprint" ""
+			(at 90.17 100.33 0)
+			(effects
+				(font
+					(size 1.27 1.27)
+				)
+				(hide yes)
+			)
+		)
+		(property "Datasheet" ""
+			(at 90.17 100.33 0)
+			(effects
+				(font
+					(size 1.27 1.27)
+				)
+				(hide yes)
+			)
+		)
+		(property "Description" "Power symbol creates a global label with name \"GND\" , ground"
+			(at 90.17 100.33 0)
+			(effects
+				(font
+					(size 1.27 1.27)
+				)
+				(hide yes)
+			)
+		)
+		(pin "1"
+		)
+		(instances
+			(project "Ecran_LCD_16_02"
+				(path "/da3a0145-d0f3-4b31-b746-e8b9b9ecb582"
+					(reference "#PWR01")
 					(unit 1)
 				)
@@
 	(symbol
 		(lib_id "Device:R")
-		(at 73.66 83.82 0)
+		(at 74.93 80.01 0)
 		(unit 1)
 		(exclude_from_sim no)
@@
 		(on_board yes)
 		(dnp no)
-		(fields_autoplaced yes)
 		(property "Reference" "R1"
-			(at 76.2 82.55 0)
+			(at 75.692 74.168 0)
 			(effects
 				(font
@@
 		)
 		(property "Value" "220"
-			(at 76.2 85.09 0)
+			(at 75.692 76.708 0)
 			(effects
 				(font
@@
 		)
 		(property "Footprint" ""
-			(at 71.882 83.82 90)
+			(at 73.152 80.01 90)
 			(effects
 				(font
@@
 		)
 		(property "Datasheet" "~"
-			(at 73.66 83.82 0)
+			(at 74.93 80.01 0)
 			(effects
 				(font
@@
 		)
 		(property "Description" ""
-			(at 73.66 83.82 0)
-			(effects
-				(font
+			(at 74.93 80.01 0)
+			(effects
+				(font
