File: 7.0/projects/Pont_H_Montage_L298N-SANS-BOUTON/Pont_H_Montage_bouttons_L298N.kicad_sch (KiCad schematic)
At the start: 26 parts, among them U1 L298N, U2 L7805

Commit message: info
Parts:
- added M1: Motor_DC, symbol Motor:Motor_DC
- added V_EXTERNE1: 5VDC, symbol Simulation_SPICE:VDC
Connections:
- net GND: now also V_EXTERNE1.2
- net VS: now also V_EXTERNE1.1
- net at D2.2 (A), D6.1 (K), OUT_MA1.1 (Pin_1)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: now also M1.1 (+)
- net at D3.2 (A), D7.1 (K), OUT_MA1.2 (Pin_2)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: now also M1.2 (-)
Other:
- moved on the sheet: ANTIHORAIRE2, C1, C2, CONTROL_INPUTS_1, CONTROL_INPUTS_2, D1, D2, D3, D4, D5, D6, D7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
