File: 7.0/projects/commande_motteur_transistor_npn/command_moteur_transistor_npn/command_moteur_transistor_npn.kicad_sch (KiCad schematic)
At the start: 7 parts, among them Q1 PN2222A, SW1 SW_Push

Commit message: adding npn
Parts:
- removed HORAIRE1: SW_A1, symbol Switch:SW_Push
- added D1: LED, symbol Device:LED
- added Q2: PN2222A, Package_TO_SOT_THT:TO-92_Inline, symbol Transistor_BJT:PN2222A
- added R1: R, symbol Device:R
- added R4, R5: 220, symbol Device:R
- added SW2: SW_Push, symbol Switch:SW_Push
- R3: value 10k -> 220
Connections:
- net GND: now also R3.1, Q2.1 (E)
- net VS: now also D1.2 (A), SW2.2
- net at R3.2: now also R5.2, SW2.1
- net at D2.1 (K): now also R1.1; no longer Q1.3 (C)
- new net: Q1.3 (C), R1.2
- new net: D1.1 (K), R4.1
- new net: Q2.3 (C), R4.2
- new net: Q2.2 (B), R5.1
Other:
- note added: "CIRCUIT PUISSANCE"
- note added: "PULL DOWN INPUT"
- note added: "PULL UP INPUT"

Commit message: adding all circuits
Parts:
- D1, D2: footprint (none) -> LED_THT:LED_D5.0mm
- R1: value R -> 220; footprint (none) -> Resistor_THT:R_Axial_DIN0411_L9.9mm_D3.6mm_P7.62mm_Vertical
- R2, R3, R4, R5: footprint (none) -> Resistor_THT:R_Axial_DIN0411_L9.9mm_D3.6mm_P7.62mm_Vertical
- SW1, SW2: footprint (none) -> Connector_PinSocket_2.54mm:PinSocket_1x02_P2.54mm_Vertical
- V_EXTERNE1: footprint (none) -> Connector_PinHeader_2.54mm:PinHeader_1x02_P2.54mm_Horizontal
Changed lines of the file:
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@@
 			)
 		)
-		(property "Value" "R"
+		(property "Value" "220"
 			(at 69.85 48.26 90)
 			(effects
@@
 			)
 		)
-		(property "Footprint" ""
+		(property "Footprint" "Resistor_THT:R_Axial_DIN0411_L9.9mm_D3.6mm_P7.62mm_Vertical"
 			(at 69.85 50.292 90)
 			(effects
@@
 			)
 		)
-		(property "Footprint" ""
+		(property "Footprint" "Resistor_THT:R_Axial_DIN0411_L9.9mm_D3.6mm_P7.62mm_Vertical"
 			(at 69.85 104.902 90)
 			(effects
@@
 			)
 		)
-		(property "Footprint" ""
+		(property "Footprint" "Resistor_THT:R_Axial_DIN0411_L9.9mm_D3.6mm_P7.62mm_Vertical"
 			(at 36.068 121.92 90)
 			(effects
@@
 			)
 		)
-		(property "Footprint" ""
+		(property "Footprint" "LED_THT:LED_D5.0mm"
 			(at 83.82 106.68 0)
 			(effects
@@
 			)
 		)
-		(property "Footprint" ""
+		(property "Footprint" "Connector_PinSocket_2.54mm:PinSocket_1x02_P2.54mm_Vertical"
 			(at 29.21 107.95 0)
 			(effects
@@
 			)
 		)
-		(property "Footprint" ""
+		(property "Footprint" "LED_THT:LED_D5.0mm"
 			(at 83.82 52.07 0)
 			(effects
@@
 			)
 		)
-		(property "Footprint" ""
+		(property "Footprint" "Resistor_THT:R_Axial_DIN0411_L9.9mm_D3.6mm_P7.62mm_Vertical"
 			(at 36.068 52.07 90)
 			(effects
@@
 			)
 		)
-		(property "Footprint" ""
+		(property "Footprint" "Connector_PinHeader_2.54mm:PinHeader_1x02_P2.54mm_Horizontal"
 			(at 54.61 34.29 0)
 			(effects
@@
 			)
 		)
-		(property "Footprint" ""
+		(property "Footprint" "Resistor_THT:R_Axial_DIN0411_L9.9mm_D3.6mm_P7.62mm_Vertical"
 			(at 44.45 112.522 90)
 			(effects
@@
 			)
 		)
-		(property "Footprint" ""
+		(property "Footprint" "Connector_PinSocket_2.54mm:PinSocket_1x02_P2.54mm_Vertical"
 			(at 29.21 64.77 0)
 			(effects
