File: 7.0/projects/Regulateur_tension-7805/regulateur_tension-7805-nov-2025-DC-DC/regulateur_tension-7805-nov-2025-DC-DC.kicad_sch (KiCad schematic)
At the start: 3 parts, among them J1 Screw_Terminal_01x02, J2 Screw_Terminal_01x02, U1 L7805

Commit message: adding fuses
Parts:
- added C1, C2: 22-47uF, symbol Device:C_Polarized
- added F1: 300mA, symbol Device:Fuse
- added J3, J4: Screw_Terminal_01x02, symbol Connector:Screw_Terminal_01x02
Connections:
- net GND: now also C1.2, C2.2
- net at J2.1 (Pin_1), U1.1 (IN): now also C1.1
- net at J1.1 (Pin_1), U1.3 (OUT): now also C2.1
- new net: J3.2 (Pin_2), J4.1 (Pin_1)
- new net: F1.2, J4.2 (Pin_2)
- new net: F1.1, J3.1 (Pin_1)
Other:
- note added: "PROTECTED SOURCE OUTPUT(12/24VDC)"
- note added: "REGULATED SOURCE(5VDC)"
- note added: "SOURCE INPUT(12/24VDC)"
- moved on the sheet: J1, J2

Commit message: info
Parts:
- C1: value 22-47uF -> 0.33uF; footprint (none) -> Capacitor_THT:C_Rect_L7.0mm_W4.5mm_P5.00mm
- C2: value 22-47uF -> 0.1uF; footprint (none) -> Capacitor_THT:C_Rect_L7.0mm_W4.5mm_P5.00mm
- F1: footprint (none) -> Fuse:Fuseholder_Cylinder-5x20mm_Stelvio-Kontek_PTF78_Horizontal_Open
- J1: renamed from J2; footprint (none) -> Connector_PinHeader_2.54mm:PinHeader_1x02_P2.54mm_Vertical
- J2: renamed from J1; footprint (none) -> Connector_PinHeader_2.54mm:PinHeader_1x02_P2.54mm_Vertical
- J3, J4: footprint (none) -> Connector_PinHeader_2.54mm:PinHeader_1x02_P2.54mm_Vertical
- U1: footprint (none) -> Package_TO_SOT_THT:TO-220-3_Vertical
Connections:
- net at J3.2 (Pin_2): now also J4.2 (Pin_2); no longer J4.1 (Pin_1)
- net at F1.2: now also J4.1 (Pin_1); no longer J4.2 (Pin_2)
Changed lines of the file:
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@@
-	)
-	(symbol
-		(lib_id "Connector:Screw_Terminal_01x02")
-		(at 129.54 114.3 0)
-		(mirror x)
-		(unit 1)
-		(exclude_from_sim no)
-		(in_bom yes)
-		(on_board yes)
-		(dnp no)
-		(property "Reference" "J4"
-			(at 132.08 114.3001 0)
-			(effects
-				(font
-					(size 1.27 1.27)
-				)
-				(justify left)
-			)
-		)
-		(property "Value" "Screw_Terminal_01x02"
-			(at 132.08 111.7601 0)
-			(effects
-				(font
-					(size 1.27 1.27)
-				)
-				(justify left)
-			)
-		)
-		(property "Footprint" ""
-			(at 129.54 114.3 0)
-			(effects
-				(font
-					(size 1.27 1.27)
-				)
-				(hide yes)
-			)
-		)
-		(property "Datasheet" "~"
-			(at 129.54 114.3 0)
-			(effects
-				(font
-					(size 1.27 1.27)
-				)
-				(hide yes)
-			)
-		)
-		(property "Description" "Generic screw terminal, single row, 01x02, script generated (kicad-library-utils/schlib/autogen/connector/)"
-			(at 129.54 114.3 0)
-			(effects
-				(font
-					(size 1.27 1.27)
-				)
-				(hide yes)
-			)
-		)
-		(pin "1"
-		)
-		(pin "2"
-		)
-		(instances
-			(project "regulateur_tension-7805-nov-2025-DC-DC"
-				(path "/7666492c-6562-4a9c-814c-e25c8f8128c0"
-					(reference "J4")
-					(unit 1)
-				)
-			)
-		)
 	)
 	(symbol
@@
 			)
 		)
-		(property "Footprint" ""
+		(property "Footprint" "Package_TO_SOT_THT:TO-220-3_Vertical"
 			(at 123.825 83.82 0)
 			(effects
@@
 			)
 		)
-		(property "Value" "22-47uF"
+		(property "Value" "0.1uF"
 			(at 140.97 84.2009 0)
 			(effects
@@
 			)
 		)
-		(property "Footprint" ""
+		(property "Footprint" "Capacitor_THT:C_Rect_L7.0mm_W4.5mm_P5.00mm"
 			(at 138.1252 87.63 0)
 			(effects
@@
 			)
 		)
-		(property "Footprint" ""
+		(property "Footprint" "Connector_PinHeader_2.54mm:PinHeader_1x02_P2.54mm_Vertical"
 			(at 92.71 111.76 0)
 			(effects
@@
 				(path "/7666492c-6562-4a9c-814c-e25c8f8128c0"
 					(reference "#PWR01")
+					(unit 1)
+				)
+			)
+		)
+	)
+	(symbol
+		(lib_id "Connector:Screw_Terminal_01x02")
+		(at 129.54 111.76 0)
+		(unit 1)
+		(exclude_from_sim no)
+		(in_bom yes)
+		(on_board yes)
+		(dnp no)
+		(fields_autoplaced yes)
+		(property "Reference" "J4"
+			(at 132.08 111.7599 0)
+			(effects
+				(font
+					(size 1.27 1.27)
+				)
+				(justify left)
+			)
+		)
+		(property "Value" "Screw_Terminal_01x02"
+			(at 132.08 114.2999 0)
+			(effects
+				(font
+					(size 1.27 1.27)
+				)
+				(justify left)
+			)
+		)
+		(property "Footprint" "Connector_PinHeader_2.54mm:PinHeader_1x02_P2.54mm_Vertical"
+			(at 129.54 111.76 0)
+			(effects
+				(font
+					(size 1.27 1.27)
+				)
+				(hide yes)
+			)
+		)
+		(property "Datasheet" "~"
+			(at 129.54 111.76 0)
+			(effects
+				(font
+					(size 1.27 1.27)
+				)
+				(hide yes)
+			)
+		)
+		(property "Description" "Generic screw terminal, single row, 01x02, script generated (kicad-library-utils/schlib/autogen/connector/)"
+			(at 129.54 111.76 0)
+			(effects
+				(font
+					(size 1.27 1.27)
+				)
+				(hide yes)
+			)
+		)
+		(pin "1"
+		)
+		(pin "2"
+		)
+		(instances
+			(project "regulateur_tension-7805-nov-2025-DC-DC"
+				(path "/7666492c-6562-4a9c-814c-e25c8f8128c0"
+					(reference "J4")
 					(unit 1)
 				)
@@
 		(on_board yes)
 		(dnp no)
-		(property "Reference" "J2"
+		(property "Reference" "J1"
 			(at 85.09 80.0099 0)
 			(effects
@@
 			)
 		)
-		(property "Footprint" ""
+		(property "Footprint" "Connector_PinHeader_2.54mm:PinHeader_1x02_P2.54mm_Vertical"
 			(at 87.63 80.01 0)
 			(effects
@@
 			(project "regulateur_tension-7805-nov-2025-DC-DC"
 				(path "/7666492c-6562-4a9c-814c-e25c8f8128c0"
-					(reference "J2")
+					(reference "J1")
 					(unit 1)
 				)
@@
 		(dnp no)
 		(fields_autoplaced yes)
-		(property "Reference" "J1"
+		(property "Reference" "J2"
 			(at 162.56 80.0099 0)
 			(effects
@@
 			)
 		)
-		(property "Footprint" ""
+		(property "Footprint" "Connector_PinHeader_2.54mm:PinHeader_1x02_P2.54mm_Vertical"
 			(at 160.02 80.01 0)
 			(effects
@@
 			(project ""
 				(path "/7666492c-6562-4a9c-814c-e25c8f8128c0"
-					(reference "J1")
+					(reference "J2")
 					(unit 1)
 				)
@@
 			)
 		)
-		(property "Footprint" ""
+		(property "Footprint" "Fuse:Fuseholder_Cylinder-5x20mm_Stelvio-Kontek_PTF78_Horizontal_Open"
 			(at 110.49 113.538 90)
 			(effects
@@
 			)
 		)
-		(property "Value" "22-47uF"
+		(property "Value" "0.33uF"
 			(at 106.68 84.2009 0)
 			(effects
@@
 			)
 		)
-		(property "Footprint" ""
+		(property "Footprint" "Capacitor_THT:C_Rect_L7.0mm_W4.5mm_P5.00mm"
 			(at 103.8352 87.63 0)
 			(effects
