File: 7.0/projects/Capteur_temperature/Capteur_temperature.kicad_sch (KiCad schematic)
At the start: 13 parts, among them U1 CC56-12CGKWA, U2 LM35-LP

Commit message: adding info
Parts:
- D1: footprint (none) -> LED_THT:LED_D5.0mm
- RA1: renamed from RA; footprint (none) -> Resistor_THT:R_Axial_DIN0411_L9.9mm_D3.6mm_P12.70mm_Horizontal
- RB1: renamed from RB; footprint (none) -> Resistor_THT:R_Axial_DIN0411_L9.9mm_D3.6mm_P12.70mm_Horizontal
- RC1: renamed from RC; footprint (none) -> Resistor_THT:R_Axial_DIN0411_L9.9mm_D3.6mm_P12.70mm_Horizontal
- RD1: renamed from RD; footprint (none) -> Resistor_THT:R_Axial_DIN0411_L9.9mm_D3.6mm_P12.70mm_Horizontal
- RE1: renamed from RE; footprint (none) -> Resistor_THT:R_Axial_DIN0411_L9.9mm_D3.6mm_P12.70mm_Horizontal
- RF1: renamed from RF; footprint (none) -> Resistor_THT:R_Axial_DIN0411_L9.9mm_D3.6mm_P12.70mm_Horizontal
- RG1: renamed from RG; footprint (none) -> Resistor_THT:R_Axial_DIN0411_L9.9mm_D3.6mm_P12.70mm_Horizontal
- RLED1: renamed from RLED; footprint (none) -> Resistor_THT:R_Axial_DIN0411_L9.9mm_D3.6mm_P12.70mm_Horizontal
- R_DP1: renamed from R_DP; footprint (none) -> Resistor_THT:R_Axial_DIN0411_L9.9mm_D3.6mm_P12.70mm_Horizontal
Other:
- note added: "Montage LM35 avec Arduino et afficheur 4 chiffres"
Changed lines of the file:
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@@
 	(generator_version "9.0")
 	(paper "A4")
+	(text "Montage LM35 avec Arduino et afficheur 4 chiffres"
+		(exclude_from_sim no)
+		(at 136.906 29.972 0)
+		(effects
+			(font
+				(size 1.397 1.397)
+				(thickness 0.2794)
+				(bold yes)
+			)
+		)
+	)
 	(wire
 		(pts
@@
 		(dnp no)
 		(fields_autoplaced yes)
-		(property "Reference" "RE"
+		(property "Reference" "RE1"
 			(at 148.59 66.0399 0)
 			(effects
@@
 			)
 		)
-		(property "Footprint" ""
+		(property "Footprint" "Resistor_THT:R_Axial_DIN0411_L9.9mm_D3.6mm_P12.70mm_Horizontal"
 			(at 144.272 67.31 90)
 			(effects
@@
 			(project "Capteur_temperature"
 				(path "/ce0803b4-491a-4569-8399-67e6462a558a"
-					(reference "RE")
+					(reference "RE1")
 					(unit 1)
 				)
@@
 		(dnp no)
 		(fields_autoplaced yes)
-		(property "Reference" "RA"
+		(property "Reference" "RA1"
 			(at 118.11 66.0399 0)
 			(effects
@@
 			)
 		)
-		(property "Footprint" ""
+		(property "Footprint" "Resistor_THT:R_Axial_DIN0411_L9.9mm_D3.6mm_P12.70mm_Horizontal"
 			(at 113.792 67.31 90)
 			(effects
@@
 			(project ""
 				(path "/ce0803b4-491a-4569-8399-67e6462a558a"
-					(reference "RA")
+					(reference "RA1")
 					(unit 1)
 				)
@@
 		(dnp no)
 		(fields_autoplaced yes)
-		(property "Reference" "RG"
+		(property "Reference" "RG1"
 			(at 163.83 66.0399 0)
 			(effects
@@
 			)
 		)
-		(property "Footprint" ""
+		(property "Footprint" "Resistor_THT:R_Axial_DIN0411_L9.9mm_D3.6mm_P12.70mm_Horizontal"
 			(at 159.512 67.31 90)
 			(effects
@@
 			(project "Capteur_temperature"
 				(path "/ce0803b4-491a-4569-8399-67e6462a558a"
-					(reference "RG")
+					(reference "RG1")
 					(unit 1)
 				)
@@
 			)
 		)
-		(property "Footprint" ""
+		(property "Footprint" "LED_THT:LED_D5.0mm"
 			(at 101.6 99.06 0)
 			(effects
@@
 		(dnp no)
 		(fields_autoplaced yes)
-		(property "Reference" "RB"
+		(property "Reference" "RB1"
 			(at 125.73 66.0399 0)
 			(effects
@@
 			)
 		)
-		(property "Footprint" ""
+		(property "Footprint" "Resistor_THT:R_Axial_DIN0411_L9.9mm_D3.6mm_P12.70mm_Horizontal"
 			(at 121.412 67.31 90)
 			(effects
@@
 			(project "Capteur_temperature"
 				(path "/ce0803b4-491a-4569-8399-67e6462a558a"
-					(reference "RB")
+					(reference "RB1")
 					(unit 1)
 				)
@@
 		(dnp no)
 		(fields_autoplaced yes)
-		(property "Reference" "R_DP"
+		(property "Reference" "R_DP1"
 			(at 172.72 66.0399 0)
 			(effects
@@
 			)
 		)
-		(property "Footprint" ""
+		(property "Footprint" "Resistor_THT:R_Axial_DIN0411_L9.9mm_D3.6mm_P12.70mm_Horizontal"
 			(at 168.402 67.31 90)
 			(effects
@@
 			(project "Capteur_temperature"
 				(path "/ce0803b4-491a-4569-8399-67e6462a558a"
-					(reference "R_DP")
+					(reference "R_DP1")
 					(unit 1)
 				)
@@
 		(on_board yes)
 		(dnp no)
-		(property "Reference" "RLED"
+		(property "Reference" "RLED1"
 			(at 104.394 89.408 0)
 			(effects
@@
 			)
 		)
-		(property "Footprint" ""
+		(property "Footprint" "Resistor_THT:R_Axial_DIN0411_L9.9mm_D3.6mm_P12.70mm_Horizontal"
 			(at 99.822 91.44 90)
 			(effects
@@
 			(project "Capteur_temperature"
 				(path "/ce0803b4-491a-4569-8399-67e6462a558a"
-					(reference "RLED")
+					(reference "RLED1")
 					(unit 1)
 				)
@@
 		(dnp no)
 		(fields_autoplaced yes)
-		(property "Reference" "RD"
+		(property "Reference" "RD1"
 			(at 140.97 66.0399 0)
 			(effects
@@
 			)
 		)
-		(property "Footprint" ""
+		(property "Footprint" "Resistor_THT:R_Axial_DIN0411_L9.9mm_D3.6mm_P12.70mm_Horizontal"
 			(at 136.652 67.31 90)
 			(effects
@@
 			(project "Capteur_temperature"
 				(path "/ce0803b4-491a-4569-8399-67e6462a558a"
-					(reference "RD")
+					(reference "RD1")
 					(unit 1)
 				)
@@
 		(dnp no)
 		(fields_autoplaced yes)
-		(property "Reference" "RC"
+		(property "Reference" "RC1"
 			(at 133.35 66.0399 0)
 			(effects
@@
 			)
 		)
-		(property "Footprint" ""
+		(property "Footprint" "Resistor_THT:R_Axial_DIN0411_L9.9mm_D3.6mm_P12.70mm_Horizontal"
 			(at 129.032 67.31 90)
 			(effects
@@
 			(project "Capteur_temperature"
 				(path "/ce0803b4-491a-4569-8399-67e6462a558a"
-					(reference "RC")
+					(reference "RC1")
 					(unit 1)
 				)
@@
 		(dnp no)
 		(fields_autoplaced yes)
-		(property "Reference" "RF"
+		(property "Reference" "RF1"
 			(at 156.21 66.0399 0)
 			(effects
@@
 			)
 		)
-		(property "Footprint" ""
+		(property "Footprint" "Resistor_THT:R_Axial_DIN0411_L9.9mm_D3.6mm_P12.70mm_Horizontal"
 			(at 151.892 67.31 90)
 			(effects
@@
 			(project "Capteur_temperature"
 				(path "/ce0803b4-491a-4569-8399-67e6462a558a"
-					(reference "RF")
+					(reference "RF1")
 					(unit 1)
 				)
